File: hardware/Electrical/CADDeck_Knob/Knob.kicad_pcb (KiCad board)
At the start: 2 copper layers, 23.4 x 23.4 mm, 8 parts, among them J1 Conn_01x01_Pin, J2 Conn_01x01_Pin, J3 Conn_01x01_Pin, J4 Conn_01x01_Pin, J5 Conn_01x01_Pin, J6 Conn_01x02_Pin, J7 Conn_01x02_Pin, U1 49E

Commit message: Knob Platine hatte Fehler
Parts:
- removed U1: 49E, Package_TO_SOT_THT:TO-92S
- added U2: 49E-TO92, Hallsensor 49E:49E-TO92, B.Cu at (139.3, 98.5)
Routing:
- net Net-(J3-Pin_1): track 3.69 -> 13.4 mm, vias 0 -> 3
- net GND: track 30.7 -> 32.0 mm, vias 0 -> 1
- net Net-(J2-Pin_1): track 26.0 -> 24.9 mm, vias 1 -> 0
- net +3.3V: track 35.2 -> 35.7 mm, vias 1 -> 2
Other:
- board text added: "Vers. 3.1"
- board text removed: "Vers. 3.0"
